File: ESP32_MAX485_Schematic/ESP32_MAX485_Schem.sch (KiCad schematic (older format))
At the start: 11 parts, among them J1 Conn_01x03_Male, U1 ESP32_DOIT_Dev_Board, U2 MAX485E

Commit message: Added LEDS to firmware
Parts:
- removed R6: 120R, symbol Device:R
- added R2: 330R, symbol Device:R
- D1: renamed from D2; value LED -> BLUE_LED
- D2: renamed from D1; value LED -> RED_LED
- renumbered R2 to R3, R3 to R4, R4 to R5, R5 to R6
Connections:
- net GND: now also D1.1 (K)
- net at R6.2, U2.7 (B): no longer D1.1 (K)
- net at U1.26 (D25): now also R2.1; no longer R1.1
- net at U1.27 (D26): now also R1.1
- net at D1.2 (A): now also R2.2
- no-connect marks 30 -> 29
Other:
- note removed: "DMX Transmit\nIndicator"
- note removed: "WIFI Conn\nIndicator"
- moved on the sheet: D1, D2, R1
Changed lines of the file:
@@
 Connection ~ 7900 5200
 Wire Wire Line
-	7550 4500 7800 4500
-Wire Wire Line
 	7900 4500 7900 4900
 Wire Wire Line
 	7550 4800 8150 4800
-Wire Wire Line
-	6750 4700 6700 4700
-Wire Wire Line
-	6700 4700 6700 4600
-Wire Wire Line
-	6750 4600 6700 4600
-$Comp
-L Device:R R5
+$Comp
+L Device:R R6
 U 1 1 5F8A03A2
 P 8700 4900
-F 0 "R5" V 8493 4900 50  0000 C CNN
+F 0 "R6" V 8493 4900 50  0000 C CNN
 F 1 "10R" V 8584 4900 50  0000 C CNN
 F 2 "" V 8630 4900 50  0001 C CNN
@@
 $EndComp
 $Comp
-L Device:R R4
+L Device:R R5
 U 1 1 5F8A0A38
 P 8700 4600
-F 0 "R4" V 8493 4600 50  0000 C CNN
+F 0 "R5" V 8493 4600 50  0000 C CNN
 F 1 "10R" V 8584 4600 50  0000 C CNN
 F 2 "" V 8630 4600 50  0001 C CNN
@@
 L power:GND #PWR01
 U 1 1 5F8C155F
-P 3700 4000
-F 0 "#PWR01" H 3700 3750 50  0001 C CNN
-F 1 "GND" V 3705 3872 50  0000 R CNN
-F 2 "" H 3700 4000 50  0001 C CNN
-F 3 "" H 3700 4000 50  0001 C CNN
-	1    3700 4000
-	0    1    1    0
-$EndComp
-Wire Wire Line
-	4200 4000 4000 4000
-$Comp
-L Device:LED D1
+P 2600 4000
+F 0 "#PWR01" H 2600 3750 50  0001 C CNN
+F 1 "GND" V 2605 3872 50  0000 R CNN
+F 2 "" H 2600 4000 50  0001 C CNN
+F 3 "" H 2600 4000 50  0001 C CNN
+	1    2600 4000
+	0    1    1    0
+$EndComp
+$Comp
+L Device:LED D2
 U 1 1 5F8FAEF8
-P 3750 4600
-F 0 "D1" H 3743 4345 50  0000 C CNN
-F 1 "LED" H 3743 4436 50  0000 C CNN
-F 2 "" H 3750 4600 50  0001 C CNN
-F 3 "~" H 3750 4600 50  0001 C CNN
-	1    3750 4600
-	-1   0    0    1
+P 3300 4400
+F 0 "D2" H 3293 4145 50  0000 C CNN
+F 1 "RED_LED" H 3293 4236 50  0000 C CNN
+F 2 "" H 3300 4400 50  0001 C CNN
+F 3 "~" H 3300 4400 50  0001 C CNN
+	1    3300 4400
+	0    1    1    0
 $EndComp
 $Comp
 L Device:R R1
 U 1 1 5F8FB28E
-P 3750 4900
-F 0 "R1" V 3543 4900 50  0000 C CNN
-F 1 "330R" V 3634 4900 50  0000 C CNN
-F 2 "" V 3680 4900 50  0001 C CNN
-F 3 "~" H 3750 4900 50  0001 C CNN
-	1    3750 4900
-	0    1    1    0
-$EndComp
-Wire Wire Line
-	3900 4600 4000 4600
-Wire Wire Line
-	4000 4600 4000 4000
-Connection ~ 4000 4000
-Wire Wire Line
-	4000 4000 3700 4000
-Wire Wire Line
-	3600 4900 3450 4900
-Wire Wire Line
-	3450 4900 3450 4600
-Wire Wire Line
-	3450 4600 3600 4600
-Wire Wire Line
-	3900 4900 4200 4900
-Text Notes 3700 4400 2    50   ~ 0
-WIFI Conn\nIndicator
-$Comp
-L Device:LED D2
+P 3800 4800
+F 0 "R1" V 3593 4800 50  0000 C CNN
+F 1 "330R" V 3684 4800 50  0000 C CNN
+F 2 "" V 3730 4800 50  0001 C CNN
+F 3 "~" H 3800 4800 50  0001 C CNN
+	1    3800 4800
+	0    1    1    0
+$EndComp
+$Comp
+L Device:LED D1
 U 1 1 5F92D43E
-P 8150 4000
-F 0 "D2" H 8143 4217 50  0000 C CNN
-F 1 "LED" H 8143 4126 50  0000 C CNN
-F 2 "" H 8150 4000 50  0001 C CNN
-F 3 "~" H 8150 4000 50  0001 C CNN
-	1    8150 4000
-	1    0    0    -1
-$EndComp
-$Comp
-L Device:R R6
-U 1 1 5F92DC1D
-P 8750 4000
-F 0 "R6" V 8543 4000 50  0000 C CNN
-F 1 "120R" V 8634 4000 50  0000 C CNN
-F 2 "" V 8680 4000 50  0001 C CNN
-F 3 "~" H 8750 4000 50  0001 C CNN
-	1    8750 4000
-	0    1    1    0
-$EndComp
-Wire Wire Line
-	9050 4600 9050 4000
-Wire Wire Line
-	9050 4000 8900 4000
-Connection ~ 9050 4600
-Wire Wire Line
-	8600 4000 8300 4000
-Wire Wire Line
-	8000 4000 7800 4000
-Wire Wire Line
-	7800 4000 7800 4500
-Connection ~ 7800 4500
-Wire Wire Line
-	7800 4500 7900 4500
-Text Notes 8400 3700 2    50   ~ 0
-DMX Transmit\nIndicator
+P 2850 4400
+F 0 "D1" H 2843 4617 50  0000 C CNN
+F 1 "BLUE_LED" H 2843 4526 50  0000 C CNN
+F 2 "" H 2850 4400 50  0001 C CNN
+F 3 "~" H 2850 4400 50  0001 C CNN
+	1    2850 4400
+	0    -1   1    0
+$EndComp
 NoConn ~ 5750 5600
 NoConn ~ 5750 5500
@@
 NoConn ~ 4200 5100
 NoConn ~ 4200 5000
-NoConn ~ 4200 4800
 NoConn ~ 4200 4700
 NoConn ~ 4200 4600
@@
 	5750 4800 6750 4800
 Wire Wire Line
-	6700 4700 6050 4700
-Wire Wire Line
 	6050 4700 6050 5200
 Wire Wire Line
 	6050 5200 5750 5200
-Connection ~ 6700 4700
-$Comp
-L Device:R R3
+$Comp
+L Device:R R4
 U 1 1 5F9F2657
 P 6300 4500
-F 0 "R3" V 6093 4500 50  0000 C CNN
+F 0 "R4" V 6093 4500 50  0000 C CNN
 F 1 "1K" V 6184 4500 50  0000 C CNN
 F 2 "" V 6230 4500 50  0001 C CNN
@@
 	5850 4700 5750 4700
 $Comp
-L Device:R R2
+L Device:R R3
 U 1 1 5F9F5093
 P 6000 4000
-F 0 "R2" H 6070 4046 50  0000 L CNN
+F 0 "R3" H 6070 4046 50  0000 L CNN
 F 1 "3K3" H 6070 3955 50  0000 L CNN
 F 2 "" V 5930 4000 50  0001 C CNN
@@
 Text Notes 6100 4200 0    50   ~ 0
 Voltage Divider
+Wire Wire Line
+	7550 4500 7900 4500
+Wire Wire Line
+	4200 4800 3950 4800
+$Comp
+L Device:R R2
+U 1 1 5F9D8970
+P 3800 5100
+F 0 "R2" V 3593 5100 50  0000 C CNN
+F 1 "330R" V 3684 5100 50  0000 C CNN
+F 2 "" V 3730 5100 50  0001 C CNN
+F 3 "~" H 3800 5100 50  0001 C CNN
+	1    3800 5100
+	0    1    1    0
+$EndComp
+Wire Wire Line
+	4200 4900 4050 4900
+Wire Wire Line
+	4050 4900 4050 5100
+Wire Wire Line
+	4050 5100 3950 5100
+Wire Wire Line
+	2600 4000 2850 4000
+Wire Wire Line
+	3300 4250 3300 4000
+Connection ~ 3300 4000
+Wire Wire Line
+	3300 4000 4200 4000
+Wire Wire Line
+	2850 4250 2850 4000
+Connection ~ 2850 4000
+Wire Wire Line
+	2850 4000 3300 4000
+Wire Wire Line
+	3300 4550 3300 4800
+Wire Wire Line
+	3300 4800 3650 4800
+Wire Wire Line
+	2850 4550 2850 5100
+Wire Wire Line
+	2850 5100 3650 5100
+Wire Wire Line
+	6050 4700 6550 4700
+Wire Wire Line
+	6750 4600 6550 4600
+Wire Wire Line
+	6550 4600 6550 4700
+Connection ~ 6550 4700
+Wire Wire Line
+	6550 4700 6750 4700
 $EndSCHEMATC
